Commit message: Usa package format 2
- Fix also old package name (elfin_ethercat_driver_v3) as dependency in 
elfin_ros_control

File: elfin_description/xacro/elfin5.urdf.xacro (robot description, xacro)
@@ -131,5 +131,5 @@
       </inertial>
     </link>
-    <joint name="e${prefix}joint4" type="revolute">
+    <joint name="${prefix}joint4" type="revolute">
       <origin xyz="0.078069 -0.11342 0" rpy="${-pi} 0 0"/>
       <parent link="${prefix}link3"/>
@@ -195,5 +195,5 @@
       </inertial>
     </link>
-    <joint name="e${prefix}joint6" type="revolute">
+    <joint name="${prefix}joint6" type="revolute">
       <origin xyz="0 -0.1065 0" rpy="0 0 0"/>
       <parent link="${prefix}link5"/>
